File: schematics/slave/BMS_slave_board.sch (EAGLE design)
At the start: 66 parts, among them IC1 78L05F, IC2 ATTINY87/167AUTOMOTIVESOIC, IC3 LT1021S, IC4 78L05F, J1 AVR_SPI_PRG_6NS, Q1 BSS123, Q2 BSS123, Q3 BSS123, Q4 BSS123, U1 LMV324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

Commit message: Re-connected sense outputs to analog ins of chip.
Added a power jumber to turn off the 5vReg and the Opamps to allow for programming
Parts:
- added JP1: (no value), jumper:JP1E
Connections:
- removed net MISO: IC2.(MISO/DO/OC0A/ADC2/PCINT2)PA2, J1.1
- removed net MOSI: IC2.(MOSI/SDA/DI/ADC4/PCINT4)PA4, J1.4
- removed net N$26: J1.2
- removed net SCK: IC2.(SCK/SCL/USCK/T1/ADC5/PCINT5)PA5, J1.3
- net +3V3: now also J1.2
- net BAT-4: now also JP1.1
- net READ1: now also IC2.(MISO/DO/OC0A/ADC2/PCINT2)PA2, J1.1
- net READ3: now also IC2.(MOSI/SDA/DI/ADC4/PCINT4)PA4, J1.4
- net READ4: now also IC2.(SCK/SCL/USCK/T1/ADC5/PCINT5)PA5, J1.3
- net VDD: now also JP1.2
Changed lines of the file:
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@@
 <part name="GND28" library="supply1" deviceset="GNDIO" device=""/>
 <part name="P+8" library="supply1" deviceset="VCC" device=""/>
+<part name="+3V7" library="supply1" deviceset="+3V3" device=""/>
+<part name="JP1" library="jumper" deviceset="JP1E" device=""/>
 </parts>
 <sheets>
@@
 <instance part="+3V2" gate="G$1" x="-53.34" y="121.92"/>
 <instance part="VDD1" gate="G$1" x="-88.9" y="121.92"/>
-<instance part="VDD2" gate="G$1" x="-109.22" y="127"/>
+<instance part="VDD2" gate="G$1" x="-109.22" y="132.08"/>
 <instance part="C1" gate="G$1" x="-81.28" y="109.22"/>
 <instance part="C2" gate="G$1" x="-58.42" y="109.22"/>
@@
 <instance part="GND28" gate="G$1" x="-12.7" y="-99.06" rot="MR0"/>
 <instance part="P+8" gate="VCC" x="-55.88" y="-71.12"/>
+<instance part="+3V7" gate="G$1" x="-50.8" y="83.82"/>
+<instance part="JP1" gate="A" x="-111.76" y="121.92" rot="R90"/>
 </instances>
 <busses>
@@
 <segment>
 <label x="-109.22" y="116.84" size="1.778" layer="95" rot="R180" xref="yes"/>
-<wire x1="-109.22" y1="114.3" x2="-109.22" y2="124.46" width="0.1524" layer="91"/>
-<pinref part="VDD2" gate="G$1" pin="VDD"/>
 <pinref part="B1" gate="1" pin="P"/>
 <wire x1="-109.22" y1="114.3" x2="-104.14" y2="114.3" width="0.1524" layer="91"/>
+<pinref part="JP1" gate="A" pin="1"/>
+<wire x1="-109.22" y1="121.92" x2="-109.22" y2="114.3" width="0.1524" layer="91"/>
 </segment>
 <segment>
@@
 <junction x="154.94" y="93.98"/>
 </segment>
+<segment>
+<pinref part="IC2" gate="1" pin="(MOSI/SDA/DI/ADC4/PCINT4)PA4"/>
+<wire x1="-7.62" y1="15.24" x2="-5.08" y2="15.24" width="0.1524" layer="91"/>
+<label x="-5.08" y="15.24" size="1.778" layer="95"/>
+</segment>
+<segment>
+<pinref part="J1" gate="G$1" pin="4"/>
+<wire x1="-55.88" y1="76.2" x2="-50.8" y2="76.2" width="0.1524" layer="91"/>
+</segment>
 </net>
 <net name="READ4" class="0">
@@
 <wire x1="154.94" y1="127" x2="162.56" y2="127" width="0.1524" layer="91"/>
 <junction x="154.94" y="127"/>
+</segment>
+<segment>
+<pinref part="IC2" gate="1" pin="(SCK/SCL/USCK/T1/ADC5/PCINT5)PA5"/>
+<wire x1="-7.62" y1="17.78" x2="-5.08" y2="17.78" width="0.1524" layer="91"/>
+<label x="-5.08" y="17.78" size="1.778" layer="95"/>
+</segment>
+<segment>
+<pinref part="J1" gate="G$1" pin="3"/>
+<wire x1="-73.66" y1="76.2" x2="-78.74" y2="76.2" width="0.1524" layer="91"/>
 </segment>
 </net>
@@
 <wire x1="154.94" y1="40.64" x2="154.94" y2="22.86" width="0.1524" layer="91"/>
 <junction x="154.94" y="22.86"/>
+</segment>
+<segment>
+<pinref part="IC2" gate="1" pin="(MISO/DO/OC0A/ADC2/PCINT2)PA2"/>
+<wire x1="-7.62" y1="10.16" x2="-5.08" y2="10.16" width="0.1524" layer="91"/>
+<label x="-5.08" y="10.16" size="1.778" layer="95"/>
+</segment>
+<segment>
+<pinref part="J1" gate="G$1" pin="1"/>
+<wire x1="-73.66" y1="78.74" x2="-78.74" y2="78.74" width="0.1524" layer="91"/>
 </segment>
 </net>
@@
 <wire x1="-10.16" y1="114.3" x2="-10.16" y2="111.76" width="0.1524" layer="91"/>
 </segment>
+<segment>
+<pinref part="J1" gate="G$1" pin="2"/>
+<wire x1="-55.88" y1="78.74" x2="-50.8" y2="78.74" width="0.1524" layer="91"/>
+<pinref part="+3V7" gate="G$1" pin="+3V3"/>
+<wire x1="-50.8" y1="81.28" x2="-50.8" y2="78.74" width="0.1524" layer="91"/>
+</segment>
 </net>
 <net name="VDD" class="0">
@@
 <wire x1="139.7" y1="33.02" x2="139.7" y2="30.48" width="0.1524" layer="91"/>
 </segment>
-</net>
-<net name="MOSI" class="0">
-<segment>
-<pinref part="J1" gate="G$1" pin="4"/>
-<wire x1="-55.88" y1="76.2" x2="-50.8" y2="76.2" width="0.1524" layer="91"/>
-</segment>
-<segment>
-<pinref part="IC2" gate="1" pin="(MOSI/SDA/DI/ADC4/PCINT4)PA4"/>
-<wire x1="-7.62" y1="15.24" x2="-5.08" y2="15.24" width="0.1524" layer="91"/>
-<label x="-5.08" y="15.24" size="1.778" layer="95"/>
-</segment>
-</net>
-<net name="MISO" class="0">
-<segment>
-<pinref part="J1" gate="G$1" pin="1"/>
-<wire x1="-73.66" y1="78.74" x2="-78.74" y2="78.74" width="0.1524" layer="91"/>
-</segment>
-<segment>
-<pinref part="IC2" gate="1" pin="(MISO/DO/OC0A/ADC2/PCINT2)PA2"/>
-<wire x1="-7.62" y1="10.16" x2="-5.08" y2="10.16" width="0.1524" layer="91"/>
-<label x="-5.08" y="10.16" size="1.778" layer="95"/>
-</segment>
-</net>
-<net name="SCK" class="0">
-<segment>
-<pinref part="J1" gate="G$1" pin="3"/>
-<wire x1="-73.66" y1="76.2" x2="-78.74" y2="76.2" width="0.1524" layer="91"/>
-</segment>
-<segment>
-<pinref part="IC2" gate="1" pin="(SCK/SCL/USCK/T1/ADC5/PCINT5)PA5"/>
-<wire x1="-7.62" y1="17.78" x2="-5.08" y2="17.78" width="0.1524" layer="91"/>
-<label x="-5.08" y="17.78" size="1.778" layer="95"/>
-</segment>
-</net>
-<net name="N$26" class="0">
-<segment>
-<pinref part="J1" gate="G$1" pin="2"/>
-<wire x1="-55.88" y1="78.74" x2="-50.8" y2="78.74" width="0.1524" layer="91"/>
-</segment>
-</net>
+<segment>
+<pinref part="VDD2" gate="G$1" pin="VDD"/>
+<pinref part="JP1" gate="A" pin="2"/>
+<wire x1="-109.22" y1="129.54" x2="-109.22" y2="124.46" width="0.1524" layer="91"/>
+</segment>
+</net>

Commit message: added dual optos for automatic linear enumeration
added header for the daisy chaining of the bus
Parts:
- added R40, R41, R42, R43: (no value), rcl:R-US_R0603
- added X1, X2: 87438-04, con-molex:87438-04
- U$1, U$2: value LTV-817 -> LTV-827; device EVT-Eagle-Library:LTV-817 -> EVT-Eagle-Library:LTV-827
Connections:
- removed net N$23: IC2.(PCINT13/ADC8/OC1BW/XTAL2/CLKO)PB5
- removed net N$24: IC2.(PCINT14/ADC9/OC1AX/INT0)PB6
- new net ENUMI: IC2.(PCINT14/ADC9/OC1AX/INT0)PB6, R43.2, U$1G$2.CO
- new net ENUMO: IC2.(PCINT13/ADC8/OC1BW/XTAL2/CLKO)PB5, R40.2
- new net IENUMI: R41.1, X2-1.S
- new net IENUMO: R42.2, U$2G$2.E, X1-1.S
- new net N$25: R40.1, U$2G$2.A
- new net N$26: R41.2, U$1G$2.CA
- net +12V: now also X1-4.S, X2-4.S
- net +5V: now also U$1G$1.E, U$1G$2.E; no longer U$1.CO
- net GND: now also R43.1, U$2G$1.CA, U$2G$2.CA; no longer U$2.CA
- net GNDIO: now also R42.1, U$1G$1.A, U$1G$2.A, X1-2.S, X2-2.S; no longer U$1.CA
- net LIN: now also X1-3.S, X2-3.S
- net N$27: now also U$2G$1.A; no longer U$2.A
- net N$29: now also U$1G$1.CA; no longer U$1.A
- net RX: now also U$1G$1.CO; no longer U$1.E
- net TXD: now also U$2G$1.E; no longer U$2.E
- net VCC: now also U$2G$1.CO, U$2G$2.CO; no longer U$2.CO
Other:
- moved on the sheet: C7, C8, IC4, R36, R37, R38, R39

Commit message: added innitial board. routed isolated LIN set dimensions
modified schematic to make certain pins more convenient
Parts:
- U$1, U$2: value LTV-827 -> LTV-827SMD; device EVT-Eagle-Library:LTV-827 -> EVT-Eagle-Library:LTV-827SMD
Connections:
- removed net N$26: R41.2, U$1G$2.CA
- new net N$23: R41.2, U$2G$1.A
- net +12V: now also X1-1.S; no longer X1-4.S
- net +5V: now also U$2G$1.CO, U$2G$2.CO; no longer U$1G$1.E, U$1G$2.E
- net ENUMI: now also U$2G$1.E; no longer U$1G$2.CO
- net GND: now also U$1G$1.CA, U$1G$2.CA; no longer U$2G$1.CA, U$2G$2.CA
- net GNDIO: now also U$2G$1.CA, U$2G$2.CA, X1-3.S; no longer U$1G$1.A, U$1G$2.A, X1-2.S
- net IENUMO: now also U$1G$1.E, X1-4.S; no longer U$2G$2.E, X1-1.S
- net LIN: now also X1-2.S; no longer X1-3.S
- net N$25: now also U$1G$1.A; no longer U$2G$2.A
- net N$27: now also U$1G$2.A; no longer U$2G$1.A
- net N$29: now also U$2G$2.A; no longer U$1G$1.CA
- net RX: now also U$2G$2.E; no longer U$1G$1.CO
- net TXD: now also U$1G$2.E; no longer U$2G$1.E
- net VCC: now also U$1G$1.CO, U$1G$2.CO; no longer U$2G$1.CO, U$2G$2.CO
Other:
- moved on the sheet: X1-1, X1-2, X1-3, X1-4
Changed lines of the file:
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@@
 <part name="P+11" library="supply1" deviceset="+12V" device=""/>
 <part name="GND33" library="supply1" deviceset="GNDIO" device=""/>
-<part name="U$1" library="EVT-Eagle-Library" deviceset="LTV-827" device=""/>
-<part name="U$2" library="EVT-Eagle-Library" deviceset="LTV-827" device=""/>
+<part name="U$1" library="EVT-Eagle-Library" deviceset="LTV-827" device="SMD"/>
+<part name="U$2" library="EVT-Eagle-Library" deviceset="LTV-827" device="SMD"/>
 </parts>
 <sheets>
@@
 <instance part="P+9" gate="1" x="215.9" y="58.42" rot="MR0"/>
 <instance part="P+10" gate="VCC" x="238.76" y="10.16"/>
-<instance part="X1" gate="-1" x="309.88" y="30.48" rot="MR180"/>
-<instance part="X1" gate="-2" x="309.88" y="33.02" rot="MR180"/>
-<instance part="X1" gate="-3" x="309.88" y="35.56" rot="MR180"/>
-<instance part="X1" gate="-4" x="309.88" y="38.1" rot="MR180"/>
+<instance part="X1" gate="-1" x="309.88" y="38.1"/>
+<instance part="X1" gate="-2" x="309.88" y="35.56"/>
+<instance part="X1" gate="-3" x="309.88" y="33.02"/>
+<instance part="X1" gate="-4" x="309.88" y="30.48"/>
 <instance part="X2" gate="-1" x="276.86" y="30.48" rot="R180"/>
 <instance part="X2" gate="-2" x="276.86" y="33.02" rot="R180"/>
@@
 <instance part="P+11" gate="1" x="287.02" y="45.72"/>
 <instance part="GND33" gate="G$1" x="287.02" y="27.94" rot="MR0"/>
-<instance part="U$1" gate="G$1" x="226.06" y="139.7" rot="R90"/>
-<instance part="U$1" gate="G$2" x="226.06" y="45.72" rot="R90"/>
-<instance part="U$2" gate="G$1" x="226.06" y="91.44" rot="R270"/>
-<instance part="U$2" gate="G$2" x="226.06" y="-2.54" rot="R270"/>
+<instance part="U$1" gate="G$2" x="226.06" y="91.44" rot="R270"/>
+<instance part="U$1" gate="G$1" x="226.06" y="-2.54" rot="R270"/>
+<instance part="U$2" gate="G$2" x="226.06" y="139.7" rot="MR270"/>
+<instance part="U$2" gate="G$1" x="226.06" y="45.72" rot="MR270"/>
 </instances>
 <busses>
@@
 <pinref part="GND23" gate="1" pin="GND"/>
 <wire x1="213.36" y1="86.36" x2="213.36" y2="83.82" width="0.1524" layer="91"/>
-<pinref part="U$2" gate="G$1" pin="CA"/>
+<pinref part="U$1" gate="G$2" pin="CA"/>
 </segment>
 <segment>
@@
 <pinref part="GND31" gate="1" pin="GND"/>
 <wire x1="213.36" y1="-7.62" x2="213.36" y2="-10.16" width="0.1524" layer="91"/>
-<pinref part="U$2" gate="G$2" pin="CA"/>
+<pinref part="U$1" gate="G$1" pin="CA"/>
 </segment>
 <segment>
@@
 <wire x1="215.9" y1="144.78" x2="215.9" y2="149.86" width="0.1524" layer="91"/>
 <pinref part="P+4" gate="1" pin="+5V"/>
-<pinref part="U$1" gate="G$1" pin="E"/>
-</segment>
-<segment>
-<wire x1="215.9" y1="50.8" x2="215.9" y2="55.88" width="0.1524" layer="91"/>
+<pinref part="U$2" gate="G$2" pin="CO"/>
+</segment>
+<segment>
 <pinref part="P+9" gate="1" pin="+5V"/>
-<pinref part="U$1" gate="G$2" pin="E"/>
+<wire x1="215.9" y1="55.88" x2="215.9" y2="50.8" width="0.1524" layer="91"/>
+<pinref part="U$2" gate="G$1" pin="CO"/>
 </segment>
 </net>
@@
 <junction x="213.36" y="134.62"/>
 <label x="208.28" y="134.62" size="1.778" layer="95" rot="R180" xref="yes"/>
-<pinref part="U$1" gate="G$1" pin="CO"/>
+<pinref part="U$2" gate="G$2" pin="E"/>
 </segment>
 </net>
@@
 <pinref part="GND21" gate="G$1" pin="GNDIO"/>
 <wire x1="241.3" y1="134.62" x2="241.3" y2="132.08" width="0.1524" layer="91"/>
-<pinref part="U$1" gate="G$1" pin="A"/>
+<pinref part="U$2" gate="G$2" pin="CA"/>
 </segment>
 <segment>
@@
 </segment>
 <segment>
-<wire x1="236.22" y1="40.64" x2="241.3" y2="40.64" width="0.1524" layer="91"/>
 <pinref part="GND29" gate="G$1" pin="GNDIO"/>
 <wire x1="241.3" y1="40.64" x2="241.3" y2="38.1" width="0.1524" layer="91"/>
-<pinref part="U$1" gate="G$2" pin="A"/>
+<wire x1="241.3" y1="40.64" x2="236.22" y2="40.64" width="0.1524" layer="91"/>
+<pinref part="U$2" gate="G$1" pin="CA"/>
 </segment>
 <segment>
@@
 <segment>
 <pinref part="X2" gate="-2" pin="S"/>
-<pinref part="X1" gate="-2" pin="S"/>
 <wire x1="279.4" y1="33.02" x2="287.02" y2="33.02" width="0.1524" layer="91"/>
 <pinref part="GND33" gate="G$1" pin="GNDIO"/>
-<wire x1="287.02" y1="33.02" x2="307.34" y2="33.02" width="0.1524" layer="91"/>
 <wire x1="287.02" y1="33.02" x2="287.02" y2="30.48" width="0.1524" layer="91"/>
+<pinref part="X1" gate="-3" pin="S"/>
+<wire x1="307.34" y1="33.02" x2="287.02" y2="33.02" width="0.1524" layer="91"/>
 <junction x="287.02" y="33.02"/>
 </segment>
@@
 <pinref part="R36" gate="G$1" pin="1"/>
 <wire x1="215.9" y1="96.52" x2="213.36" y2="96.52" width="0.1524" layer="91"/>
-<pinref part="U$2" gate="G$1" pin="A"/>
+<pinref part="U$1" gate="G$2" pin="A"/>
 </segment>
 </net>
@@
 <pinref part="R37" gate="G$1" pin="2"/>
 <wire x1="238.76" y1="144.78" x2="236.22" y2="144.78" width="0.1524" layer="91"/>
-<pinref part="U$1" gate="G$1" pin="CA"/>
+<pinref part="U$2" gate="G$2" pin="A"/>
 </segment>
 </net>
@@
 <segment>
 <pinref part="X2" gate="-4" pin="S"/>
-<pinref part="X1" gate="-4" pin="S"/>
 <wire x1="279.4" y1="38.1" x2="287.02" y2="38.1" width="0.1524" layer="91"/>
+<wire x1="287.02" y1="38.1" x2="287.02" y2="43.18" width="0.1524" layer="91"/>
+<pinref part="P+11" gate="1" pin="+12V"/>
+<pinref part="X1" gate="-1" pin="S"/>
 <wire x1="287.02" y1="38.1" x2="307.34" y2="38.1" width="0.1524" layer="91"/>
-<wire x1="287.02" y1="38.1" x2="287.02" y2="43.18" width="0.1524" layer="91"/>
 <junction x="287.02" y="38.1"/>
-<pinref part="P+11" gate="1" pin="+12V"/>
 </segment>
 </net>
@@
 <pinref part="P+8" gate="VCC" pin="VCC"/>
 <wire x1="238.76" y1="101.6" x2="238.76" y2="96.52" width="0.1524" layer="91"/>
-<pinref part="U$2" gate="G$1" pin="CO"/>
+<pinref part="U$1" gate="G$2" pin="CO"/>
 </segment>
 <segment>
@@
 <pinref part="P+10" gate="VCC" pin="VCC"/>
 <wire x1="238.76" y1="7.62" x2="238.76" y2="2.54" width="0.1524" layer="91"/>
-<pinref part="U$2" gate="G$2" pin="CO"/>
+<pinref part="U$1" gate="G$1" pin="CO"/>
 </segment>
 </net>
@@
 <junction x="238.76" y="86.36"/>
 <label x="246.38" y="86.36" size="1.778" layer="95" xref="yes"/>
-<pinref part="U$2" gate="G$1" pin="E"/>
+<pinref part="U$1" gate="G$2" pin="E"/>
 </segment>
 </net>
@@
 <segment>
 <pinref part="X2" gate="-3" pin="S"/>
-<pinref part="X1" gate="-3" pin="S"/>
 <wire x1="279.4" y1="35.56" x2="304.8" y2="35.56" width="0.1524" layer="91"/>
-<wire x1="304.8" y1="35.56" x2="307.34" y2="35.56" width="0.1524" layer="91"/>
 <wire x1="304.8" y1="35.56" x2="304.8" y2="43.18" width="0.1524" layer="91"/>
-<junction x="304.8" y="35.56"/>
 <wire x1="304.8" y1="43.18" x2="302.26" y2="43.18" width="0.1524" layer="91"/>
 <label x="302.26" y="43.18" size="1.778" layer="95" rot="R180" xref="yes"/>
+<pinref part="X1" gate="-2" pin="S"/>
+<wire x1="304.8" y1="35.56" x2="307.34" y2="35.56" width="0.1524" layer="91"/>
+<junction x="304.8" y="35.56"/>
 </segment>
 </net>
@@
 <pinref part="R40" gate="G$1" pin="1"/>
 <wire x1="215.9" y1="2.54" x2="213.36" y2="2.54" width="0.1524" layer="91"/>
-<pinref part="U$2" gate="G$2" pin="A"/>
-</segment>
-</net>
-<net name="N$26" class="0">
-<segment>
-<pinref part="R41" gate="G$1" pin="2"/>
-<wire x1="238.76" y1="50.8" x2="236.22" y2="50.8" width="0.1524" layer="91"/>
-<pinref part="U$1" gate="G$2" pin="CA"/>
+<pinref part="U$1" gate="G$1" pin="A"/>
 </segment>
 </net>
@@
 <junction x="238.76" y="-7.62"/>
 <label x="246.38" y="-7.62" size="1.778" layer="95" xref="yes"/>
-<pinref part="U$2" gate="G$2" pin="E"/>
-</segment>
-<segment>
-<pinref part="X1" gate="-1" pin="S"/>
-<wire x1="307.34" y1="30.48" x2="304.8" y2="30.48" width="0.1524" layer="91"/>
+<pinref part="U$1" gate="G$1" pin="E"/>
+</segment>
+<segment>
 <wire x1="304.8" y1="30.48" x2="304.8" y2="27.94" width="0.1524" layer="91"/>
 <label x="304.8" y="27.94" size="1.778" layer="95" rot="R270" xref="yes"/>
+<pinref part="X1" gate="-4" pin="S"/>
+<wire x1="307.34" y1="30.48" x2="304.8" y2="30.48" width="0.1524" layer="91"/>
 </segment>
 </net>
 <net name="ENUMI" class="0">
 <segment>
-<wire x1="215.9" y1="40.64" x2="213.36" y2="40.64" width="0.1524" layer="91"/>
 <pinref part="R43" gate="G$1" pin="2"/>
 <wire x1="213.36" y1="40.64" x2="213.36" y2="38.1" width="0.1524" layer="91"/>
 <wire x1="213.36" y1="40.64" x2="208.28" y2="40.64" width="0.1524" layer="91"/>
+<label x="208.28" y="40.64" size="1.778" layer="95" rot="R180" xref="yes"/>
+<wire x1="215.9" y1="40.64" x2="213.36" y2="40.64" width="0.1524" layer="91"/>
 <junction x="213.36" y="40.64"/>
-<label x="208.28" y="40.64" size="1.778" layer="95" rot="R180" xref="yes"/>
-<pinref part="U$1" gate="G$2" pin="CO"/>
+<pinref part="U$2" gate="G$1" pin="E"/>
 </segment>
 <segment>
@@
 </segment>
 </net>
+<net name="N$23" class="0">
+<segment>
+<pinref part="R41" gate="G$1" pin="2"/>
+<wire x1="238.76" y1="50.8" x2="236.22" y2="50.8" width="0.1524" layer="91"/>
+<pinref part="U$2" gate="G$1" pin="A"/>
+</segment>
+</net>

Commit message: worked on ground plane and power pour
Connections:
- net GND renamed IOGND
- net +3V3: no longer C2.1, IC1.VO, IC3.IN, J1.2
- net +5V: now also C2.1, IC1.VO, IC3.IN, J1.2
Changed lines of the file:
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@@
 <part name="R34" library="rcl" deviceset="R-US_" device="R0603"/>
 <part name="GND15" library="supply1" deviceset="GND" device=""/>
-<part name="+3V2" library="supply1" deviceset="+3V3" device=""/>
 <part name="VDD1" library="supply1" deviceset="VDD" device=""/>
 <part name="VDD2" library="supply1" deviceset="VDD" device=""/>
@@
 <part name="C3" library="resistor" deviceset="C-US" device="025-024X044"/>
 <part name="IC3" library="linear-technology" deviceset="LT1021" device="S"/>
-<part name="+3V5" library="supply1" deviceset="+3V3" device=""/>
 <part name="Q2" library="transistor-small-signal" deviceset="BSS123" device=""/>
 <part name="Q1" library="transistor-small-signal" deviceset="BSS123" device=""/>
@@
 <part name="GND28" library="supply1" deviceset="GNDIO" device=""/>
 <part name="P+8" library="supply1" deviceset="VCC" device=""/>
-<part name="+3V7" library="supply1" deviceset="+3V3" device=""/>
 <part name="JP1" library="jumper" deviceset="JP1E" device=""/>
 <part name="GND29" library="supply1" deviceset="GNDIO" device=""/>
@@
 <part name="U$1" library="EVT-Eagle-Library" deviceset="LTV-827" device="SMD"/>
 <part name="U$2" library="EVT-Eagle-Library" deviceset="LTV-827" device="SMD"/>
+<part name="P+12" library="supply1" deviceset="+5V" device=""/>
+<part name="P+13" library="supply1" deviceset="+5V" device=""/>
+<part name="P+14" library="supply1" deviceset="+5V" device=""/>
 </parts>
 <sheets>
@@
 <instance part="R34" gate="G$1" x="142.24" y="40.64"/>
 <instance part="GND15" gate="1" x="-71.12" y="99.06"/>
-<instance part="+3V2" gate="G$1" x="-53.34" y="121.92"/>
 <instance part="VDD1" gate="G$1" x="-88.9" y="121.92"/>
 <instance part="VDD2" gate="G$1" x="-109.22" y="132.08"/>
@@
 <instance part="C3" gate="G$1" x="-40.64" y="109.22"/>
 <instance part="IC3" gate="G$1" x="-17.78" y="71.12"/>
-<instance part="+3V5" gate="G$1" x="-30.48" y="83.82"/>
 <instance part="Q2" gate="G$1" x="76.2" y="81.28"/>
 <instance part="Q1" gate="G$1" x="76.2" y="114.3"/>
@@
 <instance part="GND28" gate="G$1" x="281.94" y="76.2" rot="MR0"/>
 <instance part="P+8" gate="VCC" x="238.76" y="104.14"/>
-<instance part="+3V7" gate="G$1" x="-50.8" y="83.82"/>
 <instance part="JP1" gate="A" x="-111.76" y="121.92" rot="R90"/>
 <instance part="GND29" gate="G$1" x="241.3" y="35.56" rot="MR0"/>
@@
 <instance part="U$2" gate="G$2" x="226.06" y="139.7" rot="MR270"/>
 <instance part="U$2" gate="G$1" x="226.06" y="45.72" rot="MR270"/>
+<instance part="P+12" gate="1" x="-30.48" y="83.82"/>
+<instance part="P+13" gate="1" x="-50.8" y="83.82"/>
+<instance part="P+14" gate="1" x="-53.34" y="121.92"/>
 </instances>
 <busses>
@@
 </segment>
 </net>
-<net name="GND" class="0">
+<net name="IOGND" class="0">
 <segment>
 <wire x1="-109.22" y1="60.96" x2="-109.22" y2="58.42" width="0.1524" layer="91"/>
@@
 <net name="+3V3" class="0">
 <segment>
-<wire x1="-60.96" y1="114.3" x2="-58.42" y2="114.3" width="0.1524" layer="91"/>
-<pinref part="+3V2" gate="G$1" pin="+3V3"/>
-<wire x1="-58.42" y1="114.3" x2="-53.34" y2="114.3" width="0.1524" layer="91"/>
-<wire x1="-53.34" y1="114.3" x2="-53.34" y2="119.38" width="0.1524" layer="91"/>
-<pinref part="C2" gate="G$1" pin="1"/>
-<wire x1="-58.42" y1="114.3" x2="-58.42" y2="111.76" width="0.1524" layer="91"/>
-<junction x="-58.42" y="114.3"/>
-<pinref part="IC1" gate="G$1" pin="VO"/>
-</segment>
-<segment>
 <pinref part="+3V3" gate="G$1" pin="+3V3"/>
 <pinref part="C4" gate="G$1" pin="1"/>
@@
 </segment>
 <segment>
-<pinref part="+3V5" gate="G$1" pin="+3V3"/>
-<wire x1="-30.48" y1="81.28" x2="-30.48" y2="73.66" width="0.1524" layer="91"/>
-<pinref part="IC3" gate="G$1" pin="IN"/>
-<wire x1="-30.48" y1="73.66" x2="-27.94" y2="73.66" width="0.1524" layer="91"/>
-</segment>
-<segment>
 <pinref part="+3V1" gate="G$1" pin="+3V3"/>
 <pinref part="C5" gate="G$1" pin="1"/>
@@
 <pinref part="C6" gate="G$1" pin="1"/>
 <wire x1="-10.16" y1="114.3" x2="-10.16" y2="111.76" width="0.1524" layer="91"/>
-</segment>
-<segment>
-<pinref part="J1" gate="G$1" pin="2"/>
-<wire x1="-55.88" y1="78.74" x2="-50.8" y2="78.74" width="0.1524" layer="91"/>
-<pinref part="+3V7" gate="G$1" pin="+3V3"/>
-<wire x1="-50.8" y1="81.28" x2="-50.8" y2="78.74" width="0.1524" layer="91"/>
 </segment>
 </net>
@@
 <pinref part="U$2" gate="G$1" pin="CO"/>
 </segment>
-</net>
+<segment>
+<wire x1="-30.48" y1="81.28" x2="-30.48" y2="73.66" width="0.1524" layer="91"/>
+<pinref part="IC3" gate="G$1" pin="IN"/>
+<wire x1="-30.48" y1="73.66" x2="-27.94" y2="73.66" width="0.1524" layer="91"/>
+<pinref part="P+12" gate="1" pin="+5V"/>
+</segment>
+<segment>
+<pinref part="J1" gate="G$1" pin="2"/>
+<wire x1="-55.88" y1="78.74" x2="-50.8" y2="78.74" width="0.1524" layer="91"/>
+<wire x1="-50.8" y1="81.28" x2="-50.8" y2="78.74" width="0.1524" layer="91"/>
+<pinref part="P+13" gate="1" pin="+5V"/>
+</segment>
+<segment>
+<wire x1="-60.96" y1="114.3" x2="-58.42" y2="114.3" width="0.1524" layer="91"/>
+<wire x1="-58.42" y1="114.3" x2="-53.34" y2="114.3" width="0.1524" layer="91"/>
+<wire x1="-53.34" y1="114.3" x2="-53.34" y2="119.38" width="0.1524" layer="91"/>
+<pinref part="C2" gate="G$1" pin="1"/>
+<wire x1="-58.42" y1="114.3" x2="-58.42" y2="111.76" width="0.1524" layer="91"/>
+<junction x="-58.42" y="114.3"/>
+<pinref part="IC1" gate="G$1" pin="VO"/>
+<pinref part="P+14" gate="1" pin="+5V"/>
+</segment>
+</net>
